Commit message: Added simulated arm control

File: software/ros_packages/rover_arm/config/rover_arm.ros2_control.xacro (robot description, xacro)
@@ -1,11 +1,16 @@
 <?xml version="1.0"?>
 <robot xmlns:xacro="http://www.ros.org/wiki/xacro">
-    <xacro:macro name="rover_arm_ros2_control" params="name initial_positions_file">
+    <xacro:macro name="rover_arm_ros2_control" params="name initial_positions_file ros2_control_hardware_type">
         <xacro:property name="initial_positions" value="${xacro.load_yaml(initial_positions_file)['initial_positions']}"/>
         <ros2_control name="${name}" type="system">
             <hardware>
+              <xacro:if value="${ros2_control_hardware_type == 'main'}">
                 <plugin>odrive_ros2_control_plugin/ODriveHardwareInterface</plugin>
-                <param name="can">can0</param>
+                <param name="can">can1</param>
                 <!-- <plugin>mock_components/GenericSystem</plugin> -->
+              </xacro:if>
+              <xacro:if value="${ros2_control_hardware_type == 'sim'}">
+                <plugin>mock_components/GenericSystem</plugin>
+              </xacro:if>
             </hardware>
             <joint name="base_joint">

File: software/ros_packages/rover_arm/config/rover_arm.urdf.xacro (robot description, xacro)
@@ -2,8 +2,9 @@
 <robot xmlns:xacro="http://www.ros.org/wiki/xacro" name="rover_arm">
     <xacro:arg name="initial_positions_file" default="initial_positions.yaml" />
+    <xacro:arg name="ros2_control_hardware_type" default="main" />
     <!-- Import rover_arm urdf file -->
     <xacro:include filename="$(find rover_arm_urdf)/urdf/rover_arm.urdf" />
     <!-- Import control_xacro -->
     <xacro:include filename="rover_arm.ros2_control.xacro" />
-    <xacro:rover_arm_ros2_control name="RealSystem" initial_positions_file="$(arg initial_positions_file)"/>
+    <xacro:rover_arm_ros2_control name="RealSystem" initial_positions_file="$(arg initial_positions_file)" ros2_control_hardware_type="$(arg ros2_control_hardware_type)"/>
 </robot>
