Commit message: working cameras and gimbal

File: software/ros_packages/rover_arm/config/rover_arm.urdf.xacro (robot description, xacro)
@@ -3,7 +3,8 @@
     <xacro:arg name="initial_positions_file" default="initial_positions.yaml" />
     <xacro:arg name="ros2_control_hardware_type" default="main" />
-    <xacro:include filename="$(find rover_urdf)/urdf/rover_body.urdf.xacro" />
+    <!-- <xacro:include filename="$(find rover_urdf)/urdf/rover_body.urdf.xacro" />
     <xacro:rover_body name="rover_body">
-    </xacro:rover_body>
+    </xacro:rover_body> -->
+    <link name="rover_base_origin"/>
     <!-- Import rover_arm urdf file -->
     <xacro:include filename="$(find rover_arm_urdf)/urdf/rover_arm.urdf.xacro" />
@@ -17,12 +18,13 @@
     <xacro:include filename="$(find realsense2_description)/urdf/_d405.urdf.xacro"/>
     <!-- Instantiate micros  -->
-    <xacro:sensor_d405 parent ="arm_gripper" name="d405" use_nominal_extrinsics="true">
+    <xacro:sensor_d405 parent ="rover_arm_gripper" name="d405" use_nominal_extrinsics="true">
         <origin xyz="0 0.04075 0.1" rpy="0 -1.3963 -1.5708"/>
     </xacro:sensor_d405>
     <!-- Chassis Depth Camera -->
     <xacro:include filename="$(find realsense2_description)/urdf/_d455.urdf.xacro"/>
-    <xacro:sensor_d455 parent="base_link" name="d455" use_nominal_extrinsics="true">
+<!--
+    <xacro:sensor_d455 parent="rover_arm_base_link" name="d455" use_nominal_extrinsics="true">
         <origin xyz="0.0889 0.13335 0.27" rpy="3.1415926536 0.2617994 0"/>
-    </xacro:sensor_d455>
+    </xacro:sensor_d455> -->
     <xacro:rover_arm_ros2_control name="RealSystem" initial_positions_file="$(arg initial_positions_file)" ros2_control_hardware_type="$(arg ros2_control_hardware_type)"/>
 </robot>

Commit message: Added camera to arm_gripper link

File: software/ros_packages/rover_arm/config/rover_arm.urdf.xacro (robot description, xacro)
@@ -7,4 +7,11 @@
     <!-- Import control_xacro -->
     <xacro:include filename="rover_arm.ros2_control.xacro" />
+    <!--Import camera-->
+    <!-- Include sensors and other links -->
+    <xacro:include filename="$(find realsense2_description)/urdf/_d405.urdf.xacro"/>
+    <!-- Instantiate micros  -->
+    <xacro:sensor_d405 parent ="arm_gripper" name="camera" use_nominal_extrinsics="true">
+        <origin xyz="0.025 0.06 0.1" rpy="0 -1.5707 0"/>
+    </xacro:sensor_d405>
     <xacro:rover_arm_ros2_control name="RealSystem" initial_positions_file="$(arg initial_positions_file)" ros2_control_hardware_type="$(arg ros2_control_hardware_type)"/>
 </robot>

Commit message: added pointcloud to rviz, added sensor config

File: software/ros_packages/rover_arm/config/rover_arm.urdf.xacro (robot description, xacro)
@@ -12,5 +12,5 @@
     <!-- Instantiate micros  -->
     <xacro:sensor_d405 parent ="arm_gripper" name="camera" use_nominal_extrinsics="true">
-        <origin xyz="0.025 0.06 0.1" rpy="0 -1.5707 0"/>
+        <origin xyz="0 0.05 0.1" rpy="-1.5707 -1.5707 0"/>
     </xacro:sensor_d405>
     <xacro:rover_arm_ros2_control name="RealSystem" initial_positions_file="$(arg initial_positions_file)" ros2_control_hardware_type="$(arg ros2_control_hardware_type)"/>

Commit message: fix camera and imu tfs

File: software/ros_packages/rover_arm/config/rover_arm.urdf.xacro (robot description, xacro)
@@ -17,5 +17,5 @@
     <xacro:include filename="$(find realsense2_description)/urdf/_d455.urdf.xacro"/>
     <xacro:sensor_d455 parent="base_link" name="d455" use_nominal_extrinsics="true">
-        <origin xyz="0.03 -0.075 -0.01" rpy="3.1415926536 0 0"/>
+        <origin xyz=".1415 -0.1778 -0.01" rpy="3.1415926536 0 0"/>
     </xacro:sensor_d455>
     <xacro:rover_arm_ros2_control name="RealSystem" initial_positions_file="$(arg initial_positions_file)" ros2_control_hardware_type="$(arg ros2_control_hardware_type)"/>

File: software/ros_packages/rover_arm_urdf/urdf/rover_arm.urdf (robot description, URDF)
Before this commit: robot rover_arm, 11 links, 10 joints
Joints:
- joint imu_joint: origin xyz=.3048 0 .1778 -> xyz=.254 .1778 0

Commit message: updating imu/d455 urdf links

File: software/ros_packages/rover_arm/config/rover_arm.urdf.xacro (robot description, xacro)
@@ -17,5 +17,5 @@
     <xacro:include filename="$(find realsense2_description)/urdf/_d455.urdf.xacro"/>
     <xacro:sensor_d455 parent="base_link" name="d455" use_nominal_extrinsics="true">
-        <origin xyz=".1415 -0.1778 -0.01" rpy="3.1415926536 0 0"/>
+        <origin xyz=".09144 0.2794 -0.01" rpy="3.1415926536 0 0"/>
     </xacro:sensor_d455>
     <xacro:rover_arm_ros2_control name="RealSystem" initial_positions_file="$(arg initial_positions_file)" ros2_control_hardware_type="$(arg ros2_control_hardware_type)"/>

File: software/ros_packages/rover_arm_urdf/urdf/rover_arm.urdf (robot description, URDF)
Before this commit: robot rover_arm, 11 links, 10 joints
Joints:
- joint imu_joint: origin xyz=.254 .1778 0 rpy=0 0 -1.5708 -> xyz=.1524 .1016 0 rpy=0 0 -1.5708

Commit message: yesterday's camera tf adjustments

File: software/ros_packages/rover_arm/config/rover_arm.urdf.xacro (robot description, xacro)
@@ -17,5 +17,5 @@
     <xacro:include filename="$(find realsense2_description)/urdf/_d455.urdf.xacro"/>
     <xacro:sensor_d455 parent="base_link" name="d455" use_nominal_extrinsics="true">
-        <origin xyz=".09144 0.2794 -0.01" rpy="3.1415926536 0 0"/>
+        <origin xyz="0.0889 0.13335 0.0635" rpy="3.1415926536 0.2617994 0"/>
     </xacro:sensor_d455>
     <xacro:rover_arm_ros2_control name="RealSystem" initial_positions_file="$(arg initial_positions_file)" ros2_control_hardware_type="$(arg ros2_control_hardware_type)"/>

Commit message: fix d455 urdf z

File: software/ros_packages/rover_arm/config/rover_arm.urdf.xacro (robot description, xacro)
@@ -17,5 +17,5 @@
     <xacro:include filename="$(find realsense2_description)/urdf/_d455.urdf.xacro"/>
     <xacro:sensor_d455 parent="base_link" name="d455" use_nominal_extrinsics="true">
-        <origin xyz="0.0889 0.13335 0.0635" rpy="3.1415926536 0.2617994 0"/>
+        <origin xyz="0.0889 0.13335 0.27" rpy="3.1415926536 0.2617994 0"/>
     </xacro:sensor_d455>
     <xacro:rover_arm_ros2_control name="RealSystem" initial_positions_file="$(arg initial_positions_file)" ros2_control_hardware_type="$(arg ros2_control_hardware_type)"/>

Commit message: funky yaml

File: software/ros_packages/rover_arm/config/rover_arm.urdf.xacro (robot description, xacro)
@@ -3,6 +3,12 @@
     <xacro:arg name="initial_positions_file" default="initial_positions.yaml" />
     <xacro:arg name="ros2_control_hardware_type" default="main" />
+    <xacro:include filename="$(find rover_urdf)/urdf/rover_body.urdf.xacro" />
+    <xacro:rover_body name="rover_body">
+    </xacro:rover_body>
     <!-- Import rover_arm urdf file -->
     <xacro:include filename="$(find rover_arm_urdf)/urdf/rover_arm.urdf" />
+    <xacro:rover_arm parent="rover_base_origin">
+        <origin xyz="0 0 0" rpy="0 0 0"/>
+    </xacro:sensor_d455>
     <!-- Import control_xacro -->
     <xacro:include filename="rover_arm.ros2_control.xacro" />
