Commit message: Clean rover_arm setup and rover_urdf clean up

File: software/ros_packages/rover_urdf/urdf/rover_urdf.urdf (robot description, URDF)
Before this commit: robot rover_arm, 9 links, 8 joints
Links:
- removed link arm_gripper
- removed link arm_link_0
- removed link arm_link_1
- removed link arm_link_2
- removed link arm_link_3
- removed link arm_link_4
- removed link base_link
- removed link jaws_link
- added link rover_arm_base_link; collision mesh filename=package://rover_arm_urdf/urdf/stl_files/base_link.stl; visual mesh filename=package://rover_arm_urdf/urdf/dae_files/base_link.dae
- added link rover_arm_elbow_pitch, mass 1; collision mesh filename=package://rover_arm_urdf/urdf/stl_files/arm_link_1.stl; visual mesh filename=package://rover_arm_urdf/urdf/dae_files/arm_link_1.dae
- added link rover_arm_elbow_roll, mass 1; collision mesh filename=package://rover_arm_urdf/urdf/stl_files/arm_link_2.stl; visual mesh filename=package://rover_arm_urdf/urdf/dae_files/arm_link_2.dae
- added link rover_arm_gripper, mass 1; collision mesh filename=package://rover_arm_urdf/urdf/stl_files/arm_1819_gripper.stl scale=0.001 0.001 0.001; visual mesh filename=package://rover_arm_urdf/urdf/dae_files/arm_gripper.dae
- added link rover_arm_jaws_link; visual cylinder length=0.01 radius=0.005
- added link rover_arm_shoulder, mass 1; collision mesh filename=package://rover_arm_urdf/urdf/stl_files/arm_link_0.stl; visual mesh filename=package://rover_arm_urdf/urdf/dae_files/arm_link_0.dae
- added link rover_arm_wrist_pitch, mass 1; collision mesh filename=package://rover_arm_urdf/urdf/stl_files/arm_link_3.stl; visual mesh filename=package://rover_arm_urdf/urdf/dae_files/arm_link_3.dae
- added link rover_arm_wrist_roll, mass 1; collision mesh filename=package://rover_arm_urdf/urdf/stl_files/arm_link_4.stl; visual mesh filename=package://rover_arm_urdf/urdf/dae_files/arm_link_4.dae
- link rover_base_origin: geometry collision mesh filename=package://rover_urdf/urdf/stl_files/rover_body.stl scale=0.001 0.001 0.001; visual mesh filename=package://rover_urdf/urdf/stl_files/rover_body.stl scale=0.001 0.001 0.001
Joints:
- removed joint base_joint
- removed joint elbow_pitch_joint
- removed joint elbow_roll_joint
- removed joint gripper_jaws
- removed joint rover_body_joint
- removed joint shoulder_joint
- removed joint wrist_pitch_joint
- removed joint wrist_roll_joint
- added joint rover_arm_base_joint: type revolute, parent rover_arm_base_link, child rover_arm_shoulder, origin xyz=0.055 0 0.087245 rpy=0 0 -1.5708, axis 0 0 -1, limit lower=-1.57079632679 upper=1.57079632679 effort=1000.0 velocity=5.5
- added joint rover_arm_body_joint: type fixed, parent rover_base_origin, child rover_arm_base_link, origin xyz=0.175735 0 0.03175 rpy=0.0 0.0 0.0
- added joint rover_arm_elbow_pitch_joint: type revolute, parent rover_arm_elbow_pitch, child rover_arm_elbow_roll, origin xyz=0.05925 0 0.501983 rpy=0 0 0, axis -1 0 0, limit lower=-3.1415926 upper=3.1415926 effort=1000.0 velocity=5.6
- added joint rover_arm_elbow_roll_joint: type revolute, parent rover_arm_elbow_roll, child rover_arm_wrist_pitch, origin xyz=0.063 0.000654 0.059505 rpy=0 0 0, axis 0 0 -1, limit lower=-3.141592653589793 upper=3.141592653589793 effort=1000.0 velocity=18.5
- added joint rover_arm_gripper_jaws: type fixed, parent rover_arm_gripper, child rover_arm_jaws_link, origin xyz=0 0 0.23 rpy=0 0 0
- added joint rover_arm_shoulder_joint: type revolute, parent rover_arm_shoulder, child rover_arm_elbow_pitch, origin xyz=0 0 0.151443 rpy=0 0 3.14159, axis -1 0 0, limit lower=-1.57079632679 upper=1.57079632679 effort=1000.0 velocity=3.5
- added joint rover_arm_wrist_pitch_joint: type revolute, parent rover_arm_wrist_pitch, child rover_arm_wrist_roll, origin xyz=-0.065 0 0.3318 rpy=0 0 0, axis -1 0 0, limit lower=-1.57079632679 upper=3.141592653589793 effort=1000.0 velocity=5.9
- added joint rover_arm_wrist_roll_joint: type continuous, parent rover_arm_wrist_roll, child rover_arm_gripper, origin xyz=-0.050 0 0.050484 rpy=0 0 0, axis 0 0 1, limit effort=1000.0 velocity=22.0
