Commit message: add lidar to urdf

File: software/ros_packages/rover_urdf/urdf/rover2_body.urdf.xacro (robot description, xacro)
@@ -76,4 +76,12 @@
         <link name="camera_left_chassis_link"/>
         <link name="camera_right_chassis_link"/>
+        <link name="unilidar_imu_initial">
+            <visual>
+            <origin rpy="0 0 0" xyz="0 0 0"/>
+            <geometry>
+                <cylinder radius="0.005" length="0.01"/>
+            </geometry>
+            </visual>
+        </link>
         <!-- Rear Bogie -->
         <link name="${name}_rear_bogie">
@@ -367,4 +375,9 @@
             <child link="imu_link"/>
             <origin rpy="-0.0556722 0.116731 -1.5708" xyz=".1524 .1016 0"/>
+        </joint>
+        <joint name="lidar_joint" type="fixed">
+            <parent link="${name}_base_origin"/>
+            <child link="unilidar_imu_initial"/>
+            <origin rpy="0 0 0" xyz=".1524 0 .37"/>
         </joint>
         <joint name="${name}_tower_joint" type="fixed">

Commit message: add autonomy urdf stuff

File: software/ros_packages/rover_urdf/urdf/rover2_body.urdf.xacro (robot description, xacro)
@@ -71,4 +71,9 @@
             </collision>
         </link>
+        <!-- KRJ TODO: namespace these and update them everywhere e.g. {name}_camera_left_chassis -->
+        <link name="$gps_link"></link>
+        <link name="$imu_link"></link>
+        <link name="camera_left_chassis"/>
+        <link name="camera_right_chassis"/>
         <!-- Rear Bogie -->
         <link name="${name}_rear_bogie">
@@ -341,4 +346,25 @@
             <parent link="${name}_base_origin"/>
             <child link="${name}_ebox"/>
+        </joint>
+        <!-- KRJ TODO: Verify that this offset is correct -->
+        <joint name="camera_left_chassis" type="fixed">
+            <parent link="{name}_base_origin"/>
+            <child link="camera1"/>
+            <origin xyz="0.419803 -0.020767 0.361924" rpy="0 0 0.785"/>
+        </joint>
+        <joint name="camera_right_chassis_joint" type="fixed">
+            <parent link="{name}_base_origin"/>
+            <child link="camera_right_chassis_link"/>
+            <origin xyz="-0.072197 -0.020767 0.361924" rpy="0 0 -0.785"/>
+        </joint>
+        <joint name="gps_joint" type="fixed">
+            <parent link="{name}_base_origin"/>
+            <child link="gps_link"/>
+            <origin xyz="-.1524 0 0"/>
+        </joint>
+        <joint name="imu_joint" type="fixed">
+            <parent link="{name}_base_origin"/>
+            <child link="imu_link"/>
+            <origin rpy="-0.0556722 0.116731 -1.5708" xyz=".1524 .1016 0"/>
         </joint>
         <joint name="${name}_tower_joint" type="fixed">

Commit message: fix my xacro mistakes

File: software/ros_packages/rover_urdf/urdf/rover2_body.urdf.xacro (robot description, xacro)
@@ -72,8 +72,8 @@
         </link>
         <!-- KRJ TODO: namespace these and update them everywhere e.g. {name}_camera_left_chassis -->
-        <link name="$gps_link"></link>
-        <link name="$imu_link"></link>
-        <link name="camera_left_chassis"/>
-        <link name="camera_right_chassis"/>
+        <link name="gps_link"/>
+        <link name="imu_link"/>
+        <link name="camera_left_chassis_link"/>
+        <link name="camera_right_chassis_link"/>
         <!-- Rear Bogie -->
         <link name="${name}_rear_bogie">
@@ -348,21 +348,21 @@
         </joint>
         <!-- KRJ TODO: Verify that this offset is correct -->
-        <joint name="camera_left_chassis" type="fixed">
-            <parent link="{name}_base_origin"/>
-            <child link="camera1"/>
+        <joint name="camera_left_chassis_joint" type="fixed">
+            <parent link="${name}_base_origin"/>
+            <child link="camera_left_chassis_link"/>
             <origin xyz="0.419803 -0.020767 0.361924" rpy="0 0 0.785"/>
         </joint>
         <joint name="camera_right_chassis_joint" type="fixed">
-            <parent link="{name}_base_origin"/>
+            <parent link="${name}_base_origin"/>
             <child link="camera_right_chassis_link"/>
             <origin xyz="-0.072197 -0.020767 0.361924" rpy="0 0 -0.785"/>
         </joint>
         <joint name="gps_joint" type="fixed">
-            <parent link="{name}_base_origin"/>
+            <parent link="${name}_base_origin"/>
             <child link="gps_link"/>
             <origin xyz="-.1524 0 0"/>
         </joint>
         <joint name="imu_joint" type="fixed">
-            <parent link="{name}_base_origin"/>
+            <parent link="${name}_base_origin"/>
             <child link="imu_link"/>
             <origin rpy="-0.0556722 0.116731 -1.5708" xyz=".1524 .1016 0"/>
@@ -534,3 +534,4 @@
         </gazebo>
     </xacro:macro>
+    <!-- <xacro:rover_body name="rover" hardware_type="main"/> -->
 </robot>

Commit message: update gps name: gps_link -> gps

File: software/ros_packages/rover_urdf/urdf/rover2_body.urdf.xacro (robot description, xacro)
@@ -72,5 +72,5 @@
         </link>
         <!-- KRJ TODO: namespace these and update them everywhere e.g. {name}_camera_left_chassis -->
-        <link name="gps_link"/>
+        <link name="gps"/>
         <link name="imu_link"/>
         <link name="camera_left_chassis_link"/>
@@ -360,5 +360,5 @@
         <joint name="gps_joint" type="fixed">
             <parent link="${name}_base_origin"/>
-            <child link="gps_link"/>
+            <child link="gps"/>
             <origin xyz="-.1524 0 0"/>
         </joint>
