Commit message: reorganized arm code to sit in base packages folder

File: software/ros_packages/rover_arm_urdf/urdf/rover_arm.urdf (robot description, URDF)
Before this commit: robot rover_arm, 7 links, 6 joints
Joints:
- joint shoulder_joint: origin xyz=0 0 0.151443 rpy=0 0 0 -> xyz=0 0 0.151443 rpy=0 0 3.14159

Commit message: Added autostart and auton control features

File: software/ros_packages/rover_arm_urdf/urdf/rover_arm.urdf (robot description, URDF)
Before this commit: robot rover_arm, 7 links, 6 joints
Joints:
- joint base_joint: limit lower=-1.57079632679 upper=1.57079632679 effort=1000.0 velocity=2.0 -> lower=-1.57079632679 upper=1.57079632679 effort=1000.0 velocity=6.0
- joint elbow_pitch_joint: limit lower=-1.57079632679 upper=1.57079632679 effort=1000.0 velocity=2.0 -> lower=-2.7925 upper=2.7925 effort=1000.0 velocity=6.0
- joint elbow_roll_joint: limit lower=-3.141592653589793 upper=3.141592653589793 effort=1000.0 velocity=2.0 -> lower=-3.141592653589793 upper=3.141592653589793 effort=1000.0 velocity=6.0
- joint shoulder_joint: limit lower=-1.57079632679 upper=1.57079632679 effort=1000.0 velocity=2.0 -> lower=-1.57079632679 upper=1.57079632679 effort=1000.0 velocity=6.0
- joint wrist_pitch_joint: limit lower=-1.57079632679 upper=3.141592653589793 effort=1000.0 velocity=2.0 -> lower=-1.57079632679 upper=3.141592653589793 effort=1000.0 velocity=6.0
- joint wrist_roll_joint: limit effort=1000.0 velocity=2.0 -> effort=1000.0 velocity=6.0

Commit message: fixed joint limit

File: software/ros_packages/rover_arm_urdf/urdf/rover_arm.urdf (robot description, URDF)
Before this commit: robot rover_arm, 7 links, 6 joints
Joints:
- joint elbow_pitch_joint: limit lower=-1.57079632679 upper=1.57079632679 effort=1000.0 velocity=2.0 -> lower=-3.1415926 upper=3.1415926 effort=1000.0 velocity=2.0

Commit message: add gps and imu to urdf

File: software/ros_packages/rover_arm_urdf/urdf/rover_arm.urdf (robot description, URDF)
Before this commit: robot rover_arm, 9 links, 8 joints
Links:
- added link gps; visual cylinder length=0.01 radius=0.005
- added link imu_link; visual cylinder length=0.01 radius=0.005
Joints:
- added joint gps_joint: type fixed, parent rover_base_origin, child gps, origin xyz=.1524 0 0
- added joint imu_joint: type fixed, parent rover_base_origin, child imu_link, origin xyz=.3048 0 .1778

Commit message: fix gps urdf offset

File: software/ros_packages/rover_arm_urdf/urdf/rover_arm.urdf (robot description, URDF)
Before this commit: robot rover_arm, 11 links, 10 joints
Joints:
- joint gps_joint: origin xyz=.1524 0 0 -> xyz=-.1524 0 0

Commit message: fix imu urdf orientation

File: software/ros_packages/rover_arm_urdf/urdf/rover_arm.urdf (robot description, URDF)
Before this commit: robot rover_arm, 11 links, 10 joints
Joints:
- joint imu_joint: origin xyz=.254 .1778 0 -> xyz=.254 .1778 0 rpy=0 0 -1.5708

Commit message: add lidar to urdf

File: software/ros_packages/rover_arm_urdf/urdf/rover_arm.urdf (robot description, URDF)
Before this commit: robot rover_arm, 11 links, 10 joints
Links:
- added link unilidar_imu_initial; visual cylinder length=0.01 radius=0.005
Joints:
- added joint lidar_joint: type fixed, parent rover_base_origin, child unilidar_imu_initial, origin xyz=.1524 0 .37 rpy=0 0 0

Commit message: working architecture, wrong tf for object investigation localization

File: software/ros_packages/rover_arm_urdf/urdf/rover_arm.urdf (robot description, URDF)
Before this commit: robot rover_arm, 12 links, 11 joints
Links:
- added link camera_left_chassis; visual box size=0.02 0.02 0.02
- added link camera_right_chassis; visual box size=0.02 0.02 0.02
Joints:
- added joint camera_left_joint: type fixed, parent rover_base_origin, child camera_left_chassis, origin xyz=0.1524 0.2413 0.2286 rpy=0 0 0.698
- added joint camera_right_joint: type fixed, parent rover_base_origin, child camera_right_chassis, origin xyz=0.1524 -0.2413 0.2286 rpy=0 0 -0.698
