Commit message: fixed joint axes

File: software/ros_packages/rover_arm_urdf/urdf/northrop_arm.urdf.xacro (robot description, xacro)
@@ -179,5 +179,5 @@
       <parent link="${name}_base_link"/>
       <child link="${name}_shoulder"/>
-      <axis xyz="0.0 0.0 -1.0"/>
+      <axis xyz="0.0 0.0 1.0"/>
       <limit upper="6.283185" lower="-6.283185" effort="100" velocity="1.863787"/>
     </joint>
@@ -186,5 +186,5 @@
       <parent link="${name}_shoulder"/>
       <child link="${name}_long_arm"/>
-      <axis xyz="1.0 0.0 0.0"/>
+      <axis xyz="-1.0 0.0 0.0"/>
       <limit upper="6.283185" lower="-6.283185" effort="100" velocity="0.879645"/>
     </joint>
@@ -193,5 +193,5 @@
       <parent link="${name}_long_arm"/>
       <child link="${name}_elbow_roll"/>
-      <axis xyz="-1.0 -0.0 -0.0"/>
+      <axis xyz="1.0 -0.0 -0.0"/>
       <limit upper="6.283185" lower="-6.283185" effort="100" velocity="1.310805"/>
     </joint>
@@ -200,5 +200,5 @@
       <parent link="${name}_elbow_roll"/>
       <child link="${name}_short_arm"/>
-      <axis xyz="1.0 0.0 0.0"/>
+      <axis xyz="-1.0 0.0 0.0"/>
       <limit upper="6.283185" lower="-6.283185" effort="100" velocity="1.779038"/>
     </joint>
@@ -207,5 +207,5 @@
       <parent link="${name}_short_arm"/>
       <child link="${name}_wrist_roll"/>
-      <axis xyz="-0.0 -0.0 -1.0"/>
+      <axis xyz="-0.0 -0.0 1.0"/>
       <limit upper="6.283185" lower="-6.283185" effort="100" velocity="1.897521"/>
     </joint>
@@ -214,5 +214,5 @@
       <parent link="${name}_wrist_roll"/>
       <child link="${name}_tool0"/>
-      <axis xyz="1.0 0.0 -0.0"/>
+      <axis xyz="-1.0 0.0 -0.0"/>
       <limit upper="6.283185" lower="-6.283185" effort="100" velocity="1.863787"/>
     </joint>
