Commit message: changes for northrop arm for science

File: software/ros_packages/rover_arm_urdf/urdf/northrop_arm.urdf.xacro (robot description, xacro)
@@ -148,5 +148,5 @@
         <inertia ixx="0.004268" iyy="0.006284" izz="0.003365" ixy="-0.000106" iyz="0.000102" ixz="0.00012"/>
       </inertial>
-      <visual>
+      <!-- <visual>
         <origin xyz="0.01459598 -0.05420133 -1.189494" rpy="0 0 0.097633718357"/>
         <geometry>
@@ -159,4 +159,16 @@
         <geometry>
           <mesh filename="package://rover_arm_urdf/urdf/stl_files/arm_1819_gripper.stl" scale="0.001 0.001 0.001"/>
+        </geometry>
+      </collision> -->
+      <visual>
+        <origin xyz="0 0 0.05"/>
+        <geometry>
+          <cylinder radius="0.05" length="0.1"/>
+        </geometry>
+      </visual>
+      <collision>
+        <origin xyz="0 0 0.05"/>
+        <geometry>
+          <cylinder radius="0.05" length="0.1"/>
         </geometry>
       </collision>
