Commit message: snack run

File: software/ros_packages/rover_arm_urdf/urdf/rover2_arm.urdf.xacro (robot description, xacro)
@@ -182,5 +182,5 @@
       <child link="${name}_shoulder"/>
       <axis xyz="0.0 0.0 -1.0"/>
-      <limit upper="1.570796" lower="-1.570796" effort="100" velocity="0.565478"/>
+      <limit upper="3.1416" lower="-3.1416" effort="100" velocity="0.565478"/>
     </joint>
     <joint name="${name}_shoulder_joint" type="revolute">
