Commit message: Added arm to gazebo sim

File: software/ros_packages/rover2_arm/config/rover.ros2_control.xacro (robot description, xacro)
@@ -13,5 +13,5 @@
               </xacro:if>
               <xacro:if value="${ros2_control_hardware_type == 'gazebo'}">
-                <plugin>ign_ros2_control/GazeboSystem</plugin>
+                <plugin>gz_ros2_control/GazeboSimSystem</plugin>
               </xacro:if>
             </hardware>

File: software/ros_packages/rover2_arm/config/rover.urdf.xacro (robot description, xacro)
@@ -5,9 +5,10 @@
     <xacro:arg name="drive_initial_positions_file" default="$(find rover_urdf)/ros2_control/initial_positions.yaml" />
     <xacro:arg name="attachment" default="arm" />
+    <xacro:arg name="ros2_control_config_path" default="$(find rover2_control)/config/rover_drive.yaml" />
     <xacro:property name="hardware_type" value="$(arg ros2_control_hardware_type)"/>
     <xacro:property name="front_attachment" value = "$(arg attachment)"/>
     <!-- Import rover urdf file -->
     <xacro:include filename="$(find rover_urdf)/urdf/rover2_urdf.xacro" />
-    <xacro:rover name="rover" attachment="$(arg attachment)" hardware_type="(arg ros2_control_hardware_type)"/>
+    <xacro:rover name="rover" attachment="$(arg attachment)" hardware_type="$(arg ros2_control_hardware_type)"/>
     <!-- Import control_xacro -->
     <xacro:include filename="rover.ros2_control.xacro" />
@@ -21,4 +22,4 @@
     </xacro:if>
     <!-- Include rover drive ros2_control -->
-    <xacro:rover_body_ros2_control name="rover_drive" initial_positions_file="$(arg drive_initial_positions_file)" ros2_control_hardware_type="$(arg ros2_control_hardware_type)"/>
+    <xacro:rover_body_ros2_control name="rover_drive" initial_positions_file="$(arg drive_initial_positions_file)" ros2_control_hardware_type="$(arg ros2_control_hardware_type)" controller_config_path="$(arg ros2_control_config_path)"/>
 </robot>

File: software/ros_packages/rover_urdf/ros2_control/rover_body.ros2_control.xacro (robot description, xacro)
@@ -1,5 +1,5 @@
 <?xml version="1.0"?>
 <robot xmlns:xacro="http://www.ros.org/wiki/xacro">
-    <xacro:macro name="rover_body_ros2_control" params="name initial_positions_file ros2_control_hardware_type:=main">
+    <xacro:macro name="rover_body_ros2_control" params="name initial_positions_file ros2_control_hardware_type:=main controller_config_path:='$(find rover2_control)/config/rover_drive.yaml'">
         <xacro:property name="initial_positions" value="${xacro.load_yaml(initial_positions_file)['initial_positions']}"/>
         <ros2_control name="${name}" type="system">
@@ -144,5 +144,5 @@
         <gazebo>
             <plugin filename="libgz_ros2_control-system.so" name="gz_ros2_control::GazeboSimROS2ControlPlugin">
-                <parameters>$(find rover2_control)/config/rover_drive.yaml</parameters>
+                <parameters>${controller_config_path}</parameters>
             </plugin>
         </gazebo>

File: software/ros_packages/rover_urdf/urdf/rover2_urdf.xacro (robot description, xacro)
@@ -24,4 +24,36 @@
                 <origin xyz="-0.001611 -0.040711 0.099525" rpy="0.0 -1.3963635 1.5707963"/>
             </xacro:sensor_d405>
+            <gazebo reference="d405_depth_frame">
+                <sensor name="d405" type="rgbd_camera">
+                    <ignition_frame_id>d405_depth_frame</ignition_frame_id>
+                    <camera name="d405">
+                        <horizontal_fov>1.518436</horizontal_fov>
+                        <image>
+                            <width>1280</width>
+                            <height>720</height>
+                            <format>R_FLOAT32</format>
+                        </image>
+                        <clip>
+                            <near>0.1</near>
+                            <far>10</far>
+                        </clip>
+                        <depth_camera>
+                            <clip>
+                                <near>0.2</near>
+                                <far>6</far>
+                            </clip>
+                        </depth_camera>
+                        <noise>
+                            <type>gaussian</type>
+                            <mean>0</mean>
+                            <stddev>0.01</stddev>
+                        </noise>
+                    </camera>
+                    <always_on>1</always_on>
+                    <update_rate>15</update_rate>
+                    <visualize>true</visualize>
+                    <topic>/camera/d405/depth/color</topic>
+                </sensor>
+            </gazebo>
         </xacro:if>
         <xacro:if value="${attachment== 'northrop_arm'}">
