Commit message: Correct joint limits for northrop arm

File: software/ros_packages/rover2_arm/config/rover.urdf.xacro (robot description, xacro)
@@ -19,5 +19,5 @@
     </xacro:if>
     <xacro:if value="${front_attachment == 'northrop_arm'}">
-        <xacro:rover_ros2_control name="rover_arm" initial_positions_file="$(arg initial_positions_file)" ros2_control_hardware_type="$(arg ros2_control_hardware_type)"/>
+        <xacro:rover_ros2_control name="rover_arm" initial_positions_file="$(arg initial_positions_file)" ros2_control_hardware_type="$(arg ros2_control_hardware_type)" attachment="northrop_arm"/>
     </xacro:if>
     <!-- Include rover drive ros2_control -->

File: software/ros_packages/rover_arm_urdf/urdf/northrop_arm.urdf.xacro (robot description, xacro)
@@ -180,5 +180,5 @@
       <child link="${name}_shoulder"/>
       <axis xyz="0.0 0.0 -1.0"/>
-      <limit upper="6.283185" lower="-6.283185" effort="100" velocity="1.75"/>
+      <limit upper="6.283185" lower="-6.283185" effort="100" velocity="1.863787"/>
     </joint>
     <joint name="${name}_shoulder_joint" type="revolute">
@@ -187,5 +187,5 @@
       <child link="${name}_long_arm"/>
       <axis xyz="1.0 0.0 0.0"/>
-      <limit upper="6.283185" lower="-6.283185" effort="100" velocity="0.879"/>
+      <limit upper="6.283185" lower="-6.283185" effort="100" velocity="0.879645"/>
     </joint>
     <joint name="${name}_elbow_pitch_joint" type="revolute">
@@ -194,5 +194,5 @@
       <child link="${name}_elbow_roll"/>
       <axis xyz="-1.0 -0.0 -0.0"/>
-      <limit upper="6.283185" lower="-6.283185" effort="100" velocity="1.22"/>
+      <limit upper="6.283185" lower="-6.283185" effort="100" velocity="1.310805"/>
     </joint>
     <joint name="${name}_elbow_roll_joint" type="revolute">
@@ -201,5 +201,5 @@
       <child link="${name}_short_arm"/>
       <axis xyz="1.0 0.0 0.0"/>
-      <limit upper="6.283185" lower="-6.283185" effort="100" velocity="1.65"/>
+      <limit upper="6.283185" lower="-6.283185" effort="100" velocity="1.779038"/>
     </joint>
     <joint name="${name}_wrist_pitch_joint" type="revolute">
@@ -208,5 +208,5 @@
       <child link="${name}_wrist_roll"/>
       <axis xyz="-0.0 -0.0 -1.0"/>
-      <limit upper="6.283185" lower="-6.283185" effort="100" velocity="1.75"/>
+      <limit upper="6.283185" lower="-6.283185" effort="100" velocity="1.897521"/>
     </joint>
     <joint name="${name}_wrist_roll_joint" type="revolute">
@@ -215,5 +215,5 @@
       <child link="${name}_tool0"/>
       <axis xyz="1.0 0.0 -0.0"/>
-      <limit upper="6.283185" lower="-6.283185" effort="100" velocity="1.75"/>
+      <limit upper="6.283185" lower="-6.283185" effort="100" velocity="1.863787"/>
     </joint>
     <joint name="${name}_gripper_joint" type="fixed">
